File: TaylorReceiverSchem.sch (EAGLE design)
At the start: 16 parts, among them U1 TEENSY_3.1_BASIC, U2 XBEE_ADAPTER_KIT

Commit message: New and improved board design
Parts:
- removed R4, R5, R6, R7, R8: (no value), SparkFun-Resistors:RESISTORPTH-1/4W
- added C3, C4: (no value), SparkFun-Capacitors:CAPPTH1
- added D1, D2, D3: (no value), SparkFun-LED:LED5MM
- added F1: (no value), fuse:SHK20L
- added RN1: (no value), resistor-dil:8R-N
- added SW1: (no value), special:SW_DIP-4
- added U3: XBEE-1B1, SparkFun-RF:XBEE-1B1
- R1, R2, R3: device SparkFun-Resistors:RESISTORPTH-1/4W -> SparkFun-Passives:RESISTORAXIAL-0.3
- U2: value XBEE_ADAPTER_KIT -> V_REG_LDOSMD; device Nanotronics:XBEE_ADAPTER_KIT -> SparkFun-PowerIC:V_REG_LDOSMD
Connections:
- removed net N$4: U1.0/RX1/T, U2.TX
- removed net N$5: U1.1/TX1/T, U2.RX
- new net ASC: R3.1, U3.DIO5
- new net DIP1: SW1.1, U1.9/RX2/PWM
- new net DIP2: SW1.2, U1.10/TX2/PWM
- new net DIP3: SW1.3, U1.11/MOSI
- new net DIP4: SW1.4, U1.12/MISO
- new net N$15: D1.A, R1.2
- new net N$16: D2.A, R2.2
- new net N$17: D3.A, R3.2
- new net N$2: F1.1A, JP4.PWR
- new net N$3: C3.1, C4.1, U2.OUT, U3.VDD
- new net RSSI: R2.1, U3.RSSI
- new net XBEERECV: U1.0/RX1/T, U3.DOUT
- net GND: now also C3.2, C4.2, D1.C, D2.C, D3.C, SW1.5, SW1.6, SW1.7, SW1.8, U3.DIN, U3.GND; no longer U2.GND
- net N$10: now also RN1E.1; no longer R5.1
- net N$11: now also RN1F.1; no longer R6.1
- net N$12: now also RN1G.1; no longer R7.1
- net N$13: now also RN1H.1; no longer R8.1
- net N$6: now also RN1A.1; no longer R1.1
- net N$7: now also RN1B.1; no longer R2.1
- net N$8: now also RN1C.1; no longer R3.1
- net N$9: now also RN1D.1; no longer R4.1
- net STRIP1: now also RN1A.2; no longer R1.2
- net STRIP2: now also RN1B.2; no longer R2.2
- net STRIP3: now also RN1C.2; no longer R3.2
- net STRIP4: now also RN1D.2; no longer R4.2
- net STRIP5: now also RN1E.2; no longer R5.2
- net STRIP6: now also RN1F.2; no longer R6.2
- net STRIP7: now also RN1G.2; no longer R7.2
- net STRIP8: now also RN1H.2; no longer R8.2
- net VCC: now also F1.2A, R1.1, U2.EN, U2.IN; no longer JP4.PWR, U2.3V@1, U2.3V@10
Other:
- note added: "DIP Switch Circuit"
- note added: "LED Indicators"
- note added: "Must use internal pullups in Teensy"
- note added: "XBEE and Clean Power Circuit"
- moved on the sheet: C2, JP4, R1, R2, R3

Commit message: Added right angle connectors to board.
Parts:
- removed JP1, JP2, JP3: (no value), SparkFun-Connectors:M08
- added P1, P2, P3: 39-30-08_S, con-molex-mini-fit:39-30-08_S
Connections:
- removed net N$10: JP2.3, RN1E.1
- removed net N$11: JP2.1, RN1F.1
- new net N$4: P2-5.P, RN1E.1
- new net N$5: P2-2.P, RN1F.1
- net GND: now also P1-3.P, P1-7.P, P2-3.P, P2-7.P, P3-3.P, P3-7.P; no longer JP1.4, JP1.7, JP2.4, JP2.7, JP3.4, JP3.7
- net N$12: now also P3-6.P; no longer JP3.6
- net N$13: now also P3-5.P; no longer JP3.3
- net N$6: now also P1-6.P; no longer JP1.6
- net N$7: now also P1-5.P; no longer JP1.3
- net N$8: now also P1-2.P; no longer JP1.1
- net N$9: now also P2-6.P; no longer JP2.6
- net VCC: now also P1-1.P, P1-4.P, P1-8.P, P2-1.P, P2-4.P, P2-8.P, P3-4.P, P3-8.P; no longer JP1.2, JP1.5, JP1.8, JP2.2, JP2.5, JP2.8, JP3.5, JP3.8
